File: bv_PCB/bv_PCB.kicad_pcb (KiCad board)
At the start: 2 copper layers, 69.1 x 97 mm, 26 parts, among them J1 Conn_01x06_Socket, SW1 SW_Push_45deg, SW10 SW_Push_45deg, SW11 SW_Push_45deg, SW12 SW_Push_45deg, SW2 SW_Push_45deg, SW3 SW_Push_45deg, SW4 SW_Push_45deg, SW5 SW_Push_45deg, SW6 SW_Push_45deg, SW7 SW_Push_45deg, SW8 SW_Push_45deg, SW9 SW_Push_45deg, U1 MOUDLE-SEEEDUINO-XIAO

Commit message: Nearly Done with KiCAD
Parts:
- added ?: , clipboard:462f2333-586c-4cc8-b04d-9995b911b9d8, F.Cu at (145.4, 166.4)
- added D13: SK6812MINI-E, footprints:SK6812MINI-E_fixed, F.Cu at (93.3, 99.1)
- added D14: SK6812MINI-E, footprints:SK6812MINI-E_fixed, F.Cu at (113.7, 99.1)
- added D15: SK6812MINI-E, footprints:SK6812MINI-E_fixed, F.Cu at (132.7, 99.1)
- added D16: SK6812MINI-E, footprints:SK6812MINI-E_fixed, F.Cu at (94.6, 118.1)
- added D17: SK6812MINI-E, footprints:SK6812MINI-E_fixed, F.Cu at (113.7, 118.1)
- added D18: SK6812MINI-E, footprints:SK6812MINI-E_fixed, F.Cu at (132.7, 118.1)
- added D19: SK6812MINI-E, footprints:SK6812MINI-E_fixed, F.Cu at (132.7, 137.2)
- added D20: SK6812MINI-E, footprints:SK6812MINI-E_fixed, F.Cu at (113.7, 137.2)
- added D21: SK6812MINI-E, footprints:SK6812MINI-E_fixed, F.Cu at (94.6, 137.2)
- added D22: SK6812MINI-E, footprints:SK6812MINI-E_fixed, F.Cu at (94.6, 156.2)
- added D23: SK6812MINI-E, footprints:SK6812MINI-E_fixed, F.Cu at (113.7, 156.2)
- added D24: SK6812MINI-E, footprints:SK6812MINI-E_fixed, F.Cu at (132.7, 156.2)
Connections:
- J1 pad 1: /Col 0 -> unconnected-(J1-Pin_1-Pad1)
- J1 pad 2: /Col 1 -> unconnected-(J1-Pin_2-Pad2)
- J1 pad 3: /Col 2 -> unconnected-(J1-Pin_3-Pad3)
- J1 pad 4: /JST0 -> /PWR
- J1 pad 5: /JST1 -> /JST
- U1 pad 14: unconnected-(U1-5V-Pad14) -> /PWR
- U1 pad 4: /JST1 -> unconnected-(U1-PA11_A3_D3-Pad4)
- U1 pad 5: /JST0 -> unconnected-(U1-PA8_A4_D4_SDA-Pad5)
- U1 pad 6: unconnected-(U1-PA9_A5_D5_SCL-Pad6) -> /JST
- U1 pad 7: unconnected-(U1-PB08_A6_D6_TX-Pad7) -> /RGB
Routing:
- net /PWR: track 0.00 -> 310.4 mm, vias 0 -> 16
- net GND: track 29.4 -> 330.9 mm, vias 2 -> 22
- net /RGB: track 0.00 -> 71.9 mm, vias 0 -> 5
- net Net-(D13-DOUT): track 0.00 -> 65.0 mm, vias 0 -> 4
- net Net-(D15-DOUT): track 0.00 -> 60.9 mm, vias 0 -> 4
- net Net-(D23-DOUT): track 0.00 -> 50.0 mm, vias 0 -> 8
- net Net-(D22-DOUT): track 0.00 -> 45.2 mm, vias 0 -> 6
- net /Col 1: track 119.9 -> 76.1 mm, vias 1 -> 0
- net Net-(D17-DOUT): track 0.00 -> 41.6 mm, vias 0 -> 4
- net /Col 2: track 125.0 -> 85.6 mm, vias 3 -> 0
- net Net-(D16-DOUT): track 0.00 -> 39.3 mm, vias 0 -> 4
- net Net-(D14-DOUT): track 0.00 -> 39.2 mm, vias 0 -> 4
- net /Row 3: track 64.8 -> 98.1 mm, vias 0 -> 1
- net Net-(D21-DOUT): track 0.00 -> 31.0 mm, vias 0 -> 2
- net Net-(D18-DOUT): track 0.00 -> 28.8 mm, vias 0 -> 4
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