File: bv_PCB/bv_PCB.kicad_sch (KiCad schematic)
At the start: 26 parts, among them J1 Conn_01x06_Socket, SW1 SW_Push_45deg, SW10 SW_Push_45deg, SW11 SW_Push_45deg, SW12 SW_Push_45deg, SW2 SW_Push_45deg, SW3 SW_Push_45deg, SW4 SW_Push_45deg, SW5 SW_Push_45deg, SW6 SW_Push_45deg, SW7 SW_Push_45deg, SW8 SW_Push_45deg, SW9 SW_Push_45deg, U1 MOUDLE-SEEEDUINO-XIAO

Commit message: Nearly Done with KiCAD
Parts:
- added D13, D14, D15, D16, D17, D18, D19, D20, D21, D22, D23, D24: SK6812MINI-E, footprints:SK6812MINI-E_fixed, symbol SK6812MINI-E:SK6812MINI-E
Connections:
- net Col 0: no longer J1.1 (Pin_1)
- net Col 1: no longer J1.2 (Pin_2)
- net Col 2: no longer J1.3 (Pin_3)
- net GND: now also D13.3 (VSS), D14.3 (VSS), D15.3 (VSS), D16.3 (VSS), D17.3 (VSS), D18.3 (VSS), D19.3 (VSS), D20.3 (VSS), D21.3 (VSS), D22.3 (VSS), D23.3 (VSS), D24.3 (VSS)
- net PWR: now reaches U1.14 (5V)
- net PWR: now also J1.4 (Pin_4), D13.1 (VDD), D14.1 (VDD), D15.1 (VDD), D16.1 (VDD), D17.1 (VDD), D18.1 (VDD), D19.1 (VDD), D20.1 (VDD), D21.1 (VDD), D22.1 (VDD), D23.1 (VDD), D24.1 (VDD)
- net JST: now reaches U1.6 (PA9_A5_D5_SCL)
- net JST: now also J1.5 (Pin_5)
- net RGB: now reaches U1.7 (PB08_A6_D6_TX)
- net RGB: now also D13.4 (DIN)
- net JST0: no longer names the net of U1.5 (PA8_A4_D4_SDA)
- net JST0: no longer J1.4 (Pin_4)
- net JST1: no longer names the net of U1.4 (PA11_A3_D3)
- net JST1: no longer J1.5 (Pin_5)
- new net: D18.2 (DOUT), D19.4 (DIN)
- new net: D17.2 (DOUT), D18.4 (DIN)
- new net: D16.2 (DOUT), D17.4 (DIN)
- new net: D23.2 (DOUT), D24.4 (DIN)
- new net: D22.2 (DOUT), D23.4 (DIN)
- new net: D21.2 (DOUT), D22.4 (DIN)
- new net: D14.2 (DOUT), D15.4 (DIN)
- new net: D13.2 (DOUT), D14.4 (DIN)
- new net: D15.2 (DOUT), D16.4 (DIN)
- new net: D20.2 (DOUT), D21.4 (DIN)
- new net: D19.2 (DOUT), D20.4 (DIN)
